File: keyboard_pcb_projects/keyboard_pcb_projects.kicad_pcb (KiCad board)
At the start: 2 copper layers, 157 parts, among them J1 AVR-ISP-6, SW1 SW_Push_Reset, SW10 8, SW11 9, SW12 0, SW13 -, SW14 =, SW15 Backspace, SW16 Page Up, SW17 Tab, SW18 Q, SW19 W, SW20 E, SW21 R, SW22 T, SW23 Y, SW24 U, SW25 I, SW26 O, SW27 P, SW28 [, SW29 ], SW3 1, SW30 \, SW31 Page Dn, SW32 Caps Lock, SW33 A, SW34 S, SW35 D, SW36 F, SW37 G, SW38 H, SW39 J, SW4 2, SW40 K, SW41 L, SW42 ;, SW43 ', SW44 Enter, SW46 Insert, SW47 Shift Left, SW48 Z, SW49 X, SW5 3, SW50 C, SW51 V, SW52 B, SW53 N, SW54 M, SW55 ,, SW56 ., SW57 /, SW58 Shift Right, SW6 4, SW60 Up, SW61 Delete, SW62 Ctrl, SW63 Win, SW64 Alt, SW65 Space, SW66 Alt, SW67 Fn, SW68 Left, SW69 Down, SW7 5, SW70 Right, SW71 Ctrl, SW8 6, SW9 7, U1 ATmega32U4-A, Y1 Crystal_GND24_Small

Commit message: finally wired up two of the positive ends of the usb controller
Routing:
- net /USB_D_P: track 0.00 -> 5.45 mm
Changed lines of the file:
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@@
+	)
+	(segment
+		(start 194.21875 69.78125)
+		(end 194.5 69.5)
+		(width 0.2)
+		(layer "B.Cu")
+		(net "/USB_D_P")
+	)
+	(segment
+		(start 195 69.5)
+		(end 195.21875 69.71875)
+		(width 0.2)
+		(layer "B.Cu")
+		(net "/USB_D_P")
+	)
+	(segment
+		(start 194.5 69.5)
+		(end 195 69.5)
+		(width 0.2)
+		(layer "B.Cu")
+		(net "/USB_D_P")
+	)
+	(segment
+		(start 195.21875 69.71875)
+		(end 195.21875 71.8725)
+		(width 0.2)
+		(layer "B.Cu")
+		(net "/USB_D_P")
+	)
+	(segment
+		(start 194.21875 71.8725)
+		(end 194.21875 69.78125)
+		(width 0.2)
+		(layer "B.Cu")
+		(net "/USB_D_P")
 	)
 	(segment
