File: keyboard_pcb_projects/keyboard_pcb_projects.kicad_pcb (KiCad board)
At the start: 2 copper layers, 332 x 137.5 mm, 157 parts, among them J1 AVR-ISP-6, SW1 SW_Push_Reset, SW10 8, SW11 9, SW12 0, SW13 -, SW14 =, SW15 Backspace, SW16 Page Up, SW17 Tab, SW18 Q, SW19 W, SW20 E, SW21 R, SW22 T, SW23 Y, SW24 U, SW25 I, SW26 O, SW27 P, SW28 [, SW29 ], SW3 1, SW30 \, SW31 Page Dn, SW32 Caps Lock, SW33 A, SW34 S, SW35 D, SW36 F, SW37 G, SW38 H, SW39 J, SW4 2, SW40 K, SW41 L, SW42 ;, SW43 ', SW44 Enter, SW46 Insert, SW47 Shift Left, SW48 Z, SW49 X, SW5 3, SW50 C, SW51 V, SW52 B, SW53 N, SW54 M, SW55 ,, SW56 ., SW57 /, SW58 Shift Right, SW6 4, SW60 Up, SW61 Delete, SW62 Ctrl, SW63 Win, SW64 Alt, SW65 Space, SW66 Alt, SW67 Fn, SW68 Left, SW69 Down, SW7 5, SW70 Right, SW71 Ctrl, SW8 6, SW9 7, U1 ATmega32U4-A, Y1 Crystal_GND24_Small

Commit message: new board sizing
Parts:
- moved C8 8.85 mm to (216.0, 166.6)
- moved D13 8.85 mm to (279.5, 101.5)
- moved D14 8.85 mm to (298.6, 101.5)
- moved D15 8.85 mm to (327.1, 101.5)
- moved D16 8.85 mm to (355.7, 101.5)
- moved D25 8.85 mm to (231.9, 120.6)
- moved D29 8.85 mm to (308.1, 120.6)
- moved D30 8.85 mm to (331.9, 120.6)
- moved D31 8.85 mm to (355.7, 120.6)
- moved D36 8.85 mm to (160.5, 139.6)
- moved D41 8.85 mm to (255.7, 139.6)
- moved D42 8.85 mm to (274.8, 139.6)
- moved D46 8.85 mm to (355.7, 139.6)
- moved D53 8.85 mm to (208.1, 158.7)
- moved D57 8.85 mm to (284.3, 158.7)
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Other:
- board size 332 x 137.5 mm -> 335.5 x 146 mm

Commit message: Added copper padded mounting hole and exported STEP file for the board
Parts:
- added H1: MountingHole_Pad, MountingHole:MountingHole_2.2mm_M2_Pad, F.Cu at (48.0, 80.0)
- added H2: MountingHole_Pad, MountingHole:MountingHole_2.2mm_M2_Pad, F.Cu at (48.0, 200.0)
- added H3: MountingHole_Pad, MountingHole:MountingHole_2.2mm_M2_Pad, F.Cu at (160.0, 200.0)
- added H4: MountingHole_Pad, MountingHole:MountingHole_2.2mm_M2_Pad, F.Cu at (253.0, 200.0)
- added H5: MountingHole_Pad, MountingHole:MountingHole_2.2mm_M2_Pad, F.Cu at (365.0, 200.0)
- added H6: MountingHole_Pad, MountingHole:MountingHole_2.2mm_M2_Pad, F.Cu at (365.0, 80.0)
- added H7: MountingHole_Pad, MountingHole:MountingHole_2.2mm_M2_Pad, F.Cu at (253.0, 80.0)
- added H8: MountingHole_Pad, MountingHole:MountingHole_2.2mm_M2_Pad, F.Cu at (160.0, 80.0)
Routing:
- net GND: track 261.7 -> 886.6 mm, vias 9 -> 13

Commit message: Added Silkscreen decorations to the board
Parts:
- added G***: LOGO, silkscreen_logos:design_name, F.Cu at (293.0, 170.5)
- added G***: LOGO, silkscreen_logos:silkscreen_1, F.Cu at (169.1, 136.4)
- added G***: LOGO, silkscreen_logos:small_silkscreen_1_inverted, B.Cu at (164.0, 172.5)
